Commit message: 修改

File: jaka_description/urdf/zu3_camera.xacro (robot description, xacro)
@@ -269,9 +269,6 @@
     <xacro:include filename="$(find realsense_ros_gazebo)/xacro/tracker.xacro"/>
     <xacro:include filename="$(find realsense_ros_gazebo)/xacro/depthcam.xacro"/>
-    <!-- xacro:realsense_d435 sensor_name="d435" parent_link="Link_6" rate="10">
-        <origin rpy="0 -1.57 0 " xyz="0 0 0.02"/>
-    </xacro:realsense_d435-->
-    <xacro:realsense_d435 sensor_name="d435" parent_link="world" rate="10">
-        <origin rpy="0 1.57 0 " xyz="0 0.2 1.5"/>
+    <xacro:realsense_d435 sensor_name="d435" parent_link="Link_6" rate="10">
+        <origin rpy="0 0 0 " xyz="0 0 0.02"/>
     </xacro:realsense_d435>
     <gazebo>
