Commit message: 修复bug

File: jaka_description/urdf/minicobo_camera.xacro (robot description, xacro)
@@ -3,5 +3,5 @@
      Commit Version: 1.6.0-4-g7f85cfe  Build Version: 1.6.7995.38578
      For more information, please see http://wiki.ros.org/sw_urdf_exporter -->
-<robot name="jaka_minicobo">
+<robot name="jaka_minicobo" xmlns:xacro="http://www.ros.org/wiki/xacro">
 <!-- LINK -->
     <link name="world"/>
@@ -300,4 +300,12 @@
         </actuator>
     </transmission>
+    <xacro:include filename="$(find realsense_ros_gazebo)/xacro/tracker.xacro"/>
+    <xacro:include filename="$(find realsense_ros_gazebo)/xacro/depthcam.xacro"/>
+    <!-- xacro:realsense_d435 sensor_name="d435" parent_link="Link_6" rate="10">
+        <origin rpy="0 -1.57 0 " xyz="0 0 0.02"/>
+    </xacro:realsense_d435-->
+    <xacro:realsense_d435 sensor_name="d435" parent_link="world" rate="10">
+        <origin rpy="0 1.57 0 " xyz="0 0.2 1.5"/>
+    </xacro:realsense_d435>
     <!-- Gazebo Control Plugin-->
     <gazebo>

Commit message: add end model

File: jaka_description/urdf/minicobo_camera.xacro (robot description, xacro)
@@ -158,4 +158,26 @@
       <geometry>
         <mesh filename="package://jaka_description/meshes/jaka_minicobo_meshes/Link6.STL" />
+      </geometry>
+    </collision>
+  </link>
+<link name="end_link">
+    <inertial>
+      <origin xyz="0 0 0" rpy="0 0 0" />
+      <mass value="0" />
+      <inertia ixx="0" ixy="0"  ixz="0"  iyy="0"  iyz="0" izz="0" />
+    </inertial>
+    <visual>
+      <origin xyz="0 0 0"  rpy="0 0 0" />
+      <geometry>
+        <mesh  filename="package://jaka_sim_env/model/end_model/meshes/end.dae" />
+      </geometry>
+      <material name="">
+        <color rgba="1 1 1 1" />
+      </material>
+    </visual>
+    <collision>
+      <origin xyz="0 0 0" rpy="0 0 0" />
+      <geometry>
+        <mesh filename="package://jaka_sim_env/model/end_model/meshes/end.dae" />
       </geometry>
     </collision>
@@ -209,8 +231,13 @@
     <limit lower="-6.28" upper="6.28" effort="100" velocity="1.57" />
   </joint>
-<joint name="dummy_tcp_joint" type="fixed">
+  <joint name="dummy_tcp_joint" type="fixed">
         <origin xyz="0 0 0" rpy="0 0 0" />
         <parent link="Link_6" />
         <child link="dummy_tcp" />
+    </joint>
+  <joint name="end_joint" type="fixed">
+        <origin xyz="0 0 0" rpy="0 0 0" />
+        <parent link="Link_6" />
+        <child link="end_link" />
     </joint>
 	 <!-- Gazebo -->
